File: Reflow-Plate.kicad_sch (KiCad schematic)
At the start: 16 parts, among them J1 DC-005-5A-2.0, Q1 NMOS, U1 MOUDLE-SEEEDUINO-XIAO-ESP32S3, U2 AMS1117-3.3

Commit message: Suiii
Parts:
- added D3: D_Zener, symbol Device:D_Zener
- added J2: Conn_01x04_Pin, Connector_PinHeader_2.54mm:PinHeader_1x04_P2.54mm_Horizontal, symbol Connector:Conn_01x04_Pin
- C1, C4, C6: value C -> 100nF; footprint (none) -> Capacitor_SMD:C_1206_3216Metric
- C2: value C_Polarized -> 100uF; footprint (none) -> Capacitor_SMD:CP_Elec_4x4.5
- C3, C5: value C -> 22uF; footprint (none) -> Capacitor_SMD:C_1206_3216Metric
- C7: value C -> 1nF; footprint (none) -> Capacitor_SMD:C_1206_3216Metric
- Q1: footprint (none) -> Package_TO_SOT_SMD:ATPAK-2
- R3: footprint (none) -> Resistor_SMD:R_1206_3216Metric
Connections:
- net +3V3: now also J2.3 (Pin_3)
- net GNDREF: now also J2.4 (Pin_4)
- net SCL: now also J2.2 (Pin_2)
- net SDA: now also J2.1 (Pin_1)
- net VCC: now also D3.1 (K), D3.2 (A)
Other:
- note added: "OLED with I2C"
- note added: "Xiao ESP32S3 Microcontroller"
- moved on the sheet: C3, C4, C5, C6, U1
